Commit message: URDF_Robot

File: src/arabian_robot/other /full_robot.xacro (robot description, xacro)
@@ -1,13 +1,14 @@
-<!-- <?xml version="1.0" encoding="utf-8"?> -->
+<?xml version="1.0" encoding="utf-8"?>
 <!-- This URDF was automatically created by SolidWorks to URDF Exporter! Originally created by Stephen Brawner (brawner@gmail.com)
      Commit Version: 1.6.0-4-g7f85cfe  Build Version: 1.6.7995.38578
      For more information, please see http://wiki.ros.org/sw_urdf_exporter -->
-<robot
-  name="arabian_robot" >
+<!-- <?xml version="1.0"?>
+   -->
+<robot xmlns:xacro="http://www.ros.org/wiki/xacro" name="arabian_robot" >
 <!-- Add Dummy Link  -->
 <link name="base_footprint">
     <inertial>
       <origin
-        xyz="0.0 0.0 0.0"
+        xyz="0.1 0.0 0.0"
         rpy="0 0 0" />
       <mass
@@ -33,5 +34,5 @@
     <inertial>
       <origin
-        xyz="-0.00133744334022522 6.05357174165988E-07 -0.000970131886296771"
+        xyz="-0.00133744334022522 6.05357174165988E-07 -0.00970131886296771"
         rpy="0 0 0" />
       <mass
@@ -69,5 +70,5 @@
     </collision>
   </link>
-  <link
+   <!-- <link
     name="upper_Link">
     <inertial>
@@ -172,6 +173,6 @@
     <axis
       xyz="0 0 0" />
-  </joint>
-  <link
+  </joint> -->
+   <link
     name="front_right_wheel">
     <inertial>
@@ -198,5 +199,5 @@
       </geometry>
       <material
-        name="">
+        name="blue">
         <color
           rgba="0.2 0.4 0.698039215686274 1" />
@@ -251,5 +252,5 @@
       </geometry>
       <material
-        name="">
+        name="blue">
         <color
           rgba="0.2 0.4 0.698039215686274 1" />
@@ -304,5 +305,5 @@
       </geometry>
       <material
-        name="">
+        name="blue">
         <color
           rgba="0.2 0.4 0.698039215686274 1" />
@@ -357,5 +358,5 @@
       </geometry>
       <material
-        name="">
+        name="blue">
         <color
           rgba="0.2 0.4 0.698039215686274 1" />
@@ -385,5 +386,5 @@
       xyz="0 1 0" />
   </joint>
-  <link
+  <!-- <link
     name="arabian_link">
     <inertial>
@@ -469,5 +470,5 @@
   <axis
     xyz="0 0 0" />
-</joint>
+</joint> -->
   <link
     name="lidar_link">
@@ -524,5 +525,5 @@
   </joint>
 <!-- front ultrasonic Link  -->
-  <link
+  <!-- <link
   name="ultrasonic_link">
   <inertial>
@@ -576,7 +577,7 @@
   <axis
     xyz="0 0 0" />
-</joint>
+</joint> -->
 <!-- raer ultrasonic Link  -->
-<link
+ <!-- <link
 name="rear_ultrasonic">
 <inertial>
@@ -630,7 +631,7 @@
 <axis
   xyz="0 0 0" />
-</joint>
+</joint> -->
 <!-- IMU Link  -->
-<link
+ <!-- <link
 name="imu_Link">
 <inertial>
@@ -684,13 +685,13 @@
 <axis
   xyz="0 0 0" />
-</joint>
-<gazebo reference="logo">
+ </joint> -->
+<!-- <gazebo reference="logo">
   <material>testing/material</material>
-</gazebo>
+</gazebo> -->
   <!-- <xacro:sensor_d435 parent="base_link" use_nominal_extrinsics="true">
     <origin xyz="0.28252 -0.0017175 0.029009" rpy="0 -0.25 0"/>
   </xacro:sensor_d435>
    -->
-<gazebo reference="front_left_wheel">
+<!-- <gazebo reference="front_left_wheel">
   <material>Gazebo/Black</material>
 </gazebo>
@@ -703,5 +704,6 @@
 <gazebo reference="rear_right_wheel">
   <material>Gazebo/Black</material>
-</gazebo>
+</gazebo> -->
+<!--
 <gazebo reference="arabian_link">
   <material>Gazebo/Blue</material>
@@ -727,5 +729,5 @@
 <gazebo reference="rear_ultrasonic">
   <material>Gazebo/Blue</material>
-</gazebo>
+</gazebo> -->
   <gazebo>
     <plugin
@@ -763,47 +765,43 @@
         <joint_name>rear_right_wheel_joint</joint_name>
     </plugin>
-  </gazebo>
-<gazebo reference="lidar_link">
-  <sensor name="gpu_lidar" type="gpu_lidar">
-    <pose>0 0 0 0 0 0</pose>
-    <topic>scan</topic>
-    <update_rate>10</update_rate>
-    <ray>
-      <scan>
-        <horizontal>
-          <samples>640</samples>
-          <resolution>1</resolution>
-          <min_angle>-2.596263</min_angle>
-          <max_angle> 2.596263</max_angle>
-        </horizontal>
-        <vertical>
-          <samples>1</samples>
-          <resolution>1</resolution>
-          <min_angle>0</min_angle>
-          <max_angle>0</max_angle>
-        </vertical>
-      </scan>
-      <range>
-        <min>0.08</min>
-        <max>10.0</max>
-        <resolution>0.01</resolution>
-      </range>
-      <noise>
-        <type>gaussian</type>
-        <mean>0.0</mean>
-        <stddev>0.01</stddev>
-      </noise>
-    </ray>
-    <always_on>true</always_on>
-    <visualize>true</visualize>
-  </sensor>
-</gazebo>
-<gazebo>
-  <plugin
+</gazebo>
+ <gazebo>
+  <!-- <plugin
     filename="gz-sim-sensors-system"
     name="gz::sim::systems::Sensors">
     <render_engine>ogre2</render_engine>
-  </plugin>
-</gazebo>
+  </plugin> -->
+ </gazebo>
+ <gazebo reference="lidar_link">
+  <sensor name='gpu_lidar' type='gpu_lidar'>"
+    <pose relative_to='lidar_link'>0 0 0 0 0 0</pose>
+    <topic>lidar</topic>
+    <update_rate>10</update_rate>
+    <lidar>
+        <scan>
+            <horizontal>
+                <samples>640</samples>
+                <resolution>1</resolution>
+                <min_angle>-1.396263</min_angle>
+                <max_angle>1.396263</max_angle>
+            </horizontal>
+            <vertical>
+                <samples>1</samples>
+                <resolution>0.01</resolution>
+                <min_angle>0</min_angle>
+                <max_angle>0</max_angle>
+            </vertical>
+        </scan>
+        <range>
+            <min>0.08</min>
+            <max>10.0</max>
+            <resolution>0.01</resolution>
+        </range>
+    </lidar>
+    <always_on>1</always_on>
+    <visualize>true</visualize>
+</sensor>
+  </gazebo>
+<!--
 <gazebo reference="imu_Link">
 <sensor name="imu_sensor" type="imu">
@@ -818,4 +816,4 @@
         name="gz::sim::systems::Imu">
 </plugin>
-</gazebo>
+</gazebo> -->
 </robot>
